File: KiCAD/A2630-New-KiCAD-Rev410-PGA/Card Edge.kicad_sch (KiCad schematic)
At the start: 33 parts, among them CN700 Amiga-2000-CPU-Slot, U204 74AHCT04, U300 74HCT05, U700 74HCT174, U701 74FCT646, U702 74FCT646, U703 74HCT245, U704 74HCT245, U705 74HCT245, U706 74HCT245, U707 74HCT245

Commit message: Better for SMD assembly now. DRC still not done.
Parts:
- C700, C701, C702, C703, C704, C705, C706, C707: LCSC (none) -> C49678
- C712, C714, C718, C719, C720: footprint Capacitor_THT:CP_Radial_D5.0mm_P2.00mm -> Capacitor_SMD:CP_Elec_6.3x5.8; LCSC (none) -> C5246550
- C713: footprint Capacitor_THT:CP_Radial_D5.0mm_P2.00mm -> Capacitor_SMD:CP_Elec_6.3x5.8; LCSC (none) -> C5246536
- R303, R304, R305, R306, R404, R405, R706: LCSC (none) -> C17513
- U204: LCSC (none) -> C7159
- U300: LCSC (none) -> C2870691
- U700: footprint Package_SO:SOIC-16_3.9x9.9mm_P1.27mm -> Package_SO:TSSOP-16_4.4x5mm_P0.65mm; LCSC (none) -> C2677702
- U701, U702: footprint Package_SO:SOIC-24W_7.5x15.4mm_P1.27mm -> Package_SO:SSOP-24_3.9x8.7mm_P0.635mm; LCSC (none) -> C2873070
- U703, U704, U705, U706, U707: LCSC (none) -> C132267
