File: KiCAD/A2630-New-KiCAD-Rev410-PGA/Logic.kicad_sch (KiCad schematic)
At the start: 62 parts, among them CN5 ATA/IDE, CN6 LED, CN7 COMPACT FLASH ATA, J901 CF SEL, J905 CABLE SELECT, Q900 MMBT3906, U300 74HCT05, U418 74LVC245, U419 74LVC245, U420 74LVC245, U421 74LVC245, U606 74HCT244, U900 74HCT245, U901 74HCT245, U902 74HCT245

Commit message: Better for SMD assembly now. DRC still not done.
Parts:
- C300, C418, C419, C420, C421, C606, C900, C901, C902, C903: LCSC (none) -> C49678
- CN7: LCSC (none) -> C444353
- Q900: LCSC (none) -> C181120
- R300, R301, R302, R407, R408, R501, R901, R902, R904: LCSC (none) -> C17513
- R903: LCSC (none) -> C17414
- R905, R931: LCSC (none) -> C17673
- R906, R907, R908, R909, R910, R911, R912, R913, R914, R915, R916, R917, R918, R919, R920, R921, R922, R923, R925, R926, R927, R928, R929: LCSC (none) -> C17561
- R924: LCSC (none) -> C17841
- R930: LCSC (none) -> C17471
- U300: LCSC (none) -> C2870691
- U418, U419, U420, U421: LCSC (none) -> C7848
- U606: LCSC (none) -> C6776
- U900, U901, U902: LCSC (none) -> C6779
