File: KiCAD/A2630-New-KiCAD-Rev410-PGA/Processor.kicad_sch (KiCad schematic)
At the start: 60 parts, among them J202 25/FPU, U200 MC68030, U201 MC68882, U204 74AHCT04, X1 25MHz, X2 50MHz

Commit message: Better for SMD assembly now. DRC still not done.
Parts:
- removed R100, R101, R102, R103, R104, R105, R106, R131: 1K, Resistor_SMD:R_0805_2012Metric, symbol Device:R
- removed RN104, RN105, RN106, RN107, RN108, RN109, RN110: 1K, Resistor_THT:R_Array_SIP9, symbol Device:R_Network08
- added RN104, RN105, RN106, RN107, RN108, RN109, RN110, RN111, RN112, RN113, RN114, RN115, RN116, RN117, RN118, RN119: 1k, Resistor_SMD:R_Array_Convex_4x0603, symbol Device:R_Pack04
- C204: LCSC (none) -> C49678
- C210, C211, C212, C213: LCSC (none) -> C1804
- CX1, CX2: LCSC (none) -> C1710
- R203, R204, R206, R207, R209, R210, R211, R212, R213, R216, R238: LCSC (none) -> C17802
- R217, R218, R219, R220, R221, R222, R223, R224, R225: LCSC (none) -> C17513
- R226, R227: LCSC (none) -> C17513; now not fitted; now left out of the parts list
- R228, R229, R230, R231, R232, R233, R234, R235, R236, R237: LCSC (none) -> C26010
- U204: LCSC (none) -> C7159
- X1, X2: symbol N2630:CXO_DIP8 -> Oscillator:CXO_DIP8
Connections:
- net A0: now also RN113.8 (R1.2)
- net A1: now also RN113.5 (R4.2)
- net A10: now also RN112.6 (R3.2)
- net A11: now also RN112.8 (R1.2)
- net A12: now also RN112.7 (R2.2)
- net A13: now also RN115.6 (R3.2)
- net A14: now also RN115.7 (R2.2)
- net A15: now also RN115.5 (R4.2)
- net A16: now also RN116.8 (R1.2)
- net A17: now also RN116.7 (R2.2)
- net A18: now also RN116.6 (R3.2)
- net A19: now also RN116.5 (R4.2)
- net A2: now also RN113.6 (R3.2)
- net A20: now also RN117.8 (R1.2)
- net A21: now also RN117.7 (R2.2)
- net A22: now also RN117.6 (R3.2)
- net A23: now also RN117.5 (R4.2)
- net A24: now also RN118.8 (R1.2)
- net A25: now also RN118.7 (R2.2)
- net A26: now also RN118.6 (R3.2)
- net A27: now also RN118.5 (R4.2)
- net A28: now also RN119.8 (R1.2)
- net A29: now also RN119.7 (R2.2)
- net A3: now also RN113.7 (R2.2)
- net A30: now also RN119.6 (R3.2)
- net A31: now also RN119.5 (R4.2)
- net A4: now also RN114.5 (R4.2)
- net A5: now also RN114.6 (R3.2)
- net A6: now also RN114.7 (R2.2)
- net A7: now also RN114.8 (R1.2)
- net A8: now also RN115.8 (R1.2)
- net A9: now also RN112.5 (R4.2)
- net D0: now also RN104.1 (R1.1)
- net D1: now also RN104.2 (R2.1)
- net D10: now also RN106.3 (R3.1)
- net D11: now also RN106.4 (R4.1)
- net D12: now also RN107.1 (R1.1)
- net D13: now also RN107.2 (R2.1)
- net D14: now also RN107.3 (R3.1)
- net D15: now also RN107.4 (R4.1)
- net D16: now also RN108.4 (R4.1)
- net D17: now also RN108.3 (R3.1)
- net D18: now also RN108.2 (R2.1)
- net D19: now also RN108.1 (R1.1)
- net D2: now also RN105.1 (R1.1)
- net D20: now also RN109.1 (R1.1)
- net D21: now also RN109.2 (R2.1)
- net D22: now also RN109.3 (R3.1)
- net D23: now also RN109.4 (R4.1)
- net D24: now also RN110.4 (R4.1)
- net D25: now also RN110.3 (R3.1)
- net D26: now also RN110.2 (R2.1)
- net D27: now also RN110.1 (R1.1)
- net D28: now also RN111.1 (R1.1)
- net D29: now also RN111.2 (R2.1)
- net D3: now also RN104.4 (R4.1)
- net D30: now also RN111.3 (R3.1)
- net D31: now also RN111.4 (R4.1)
- net D4: now also RN104.3 (R3.1)
- net D5: now also RN105.2 (R2.1)
- net D6: now also RN105.3 (R3.1)
- net D7: now also RN105.4 (R4.1)
- net D8: now also RN106.2 (R2.1)
- net D9: now also RN106.1 (R1.1)
- net GND: now also RN104.5 (R4.2), RN104.6 (R3.2), RN104.7 (R2.2), RN104.8 (R1.2), RN105.5 (R4.2), RN105.6 (R3.2), RN105.7 (R2.2), RN105.8 (R1.2), RN106.5 (R4.2), RN106.6 (R3.2), RN106.7 (R2.2), RN106.8 (R1.2), RN107.5 (R4.2), RN107.6 (R3.2), RN107.7 (R2.2), RN107.8 (R1.2), RN108.5 (R4.2), RN108.6 (R3.2), RN108.7 (R2.2), RN108.8 (R1.2), RN109.5 (R4.2), RN109.6 (R3.2), RN109.7 (R2.2), RN109.8 (R1.2), RN110.5 (R4.2), RN110.6 (R3.2), RN110.7 (R2.2), RN110.8 (R1.2), RN111.5 (R4.2), RN111.6 (R3.2), RN111.7 (R2.2), RN111.8 (R1.2), RN112.1 (R1.1), RN112.2 (R2.1), RN112.3 (R3.1), RN112.4 (R4.1), RN113.1 (R1.1), RN113.2 (R2.1), RN113.3 (R3.1), RN113.4 (R4.1), RN114.1 (R1.1), RN114.2 (R2.1), RN114.3 (R3.1), RN114.4 (R4.1), RN115.1 (R1.1), RN115.2 (R2.1), RN115.3 (R3.1), RN115.4 (R4.1), RN116.1 (R1.1), RN116.2 (R2.1), RN116.3 (R3.1), RN116.4 (R4.1), RN117.1 (R1.1), RN117.2 (R2.1), RN117.3 (R3.1), RN117.4 (R4.1), RN118.1 (R1.1), RN118.2 (R2.1), RN118.3 (R3.1), RN118.4 (R4.1), RN119.1 (R1.1), RN119.2 (R2.1), RN119.3 (R3.1), RN119.4 (R4.1)
Other:
- moved on the sheet: X1, X2
